File: pcb/pcb/_autosave-pcb.kicad_sch (KiCad schematic)
At the start: 16 parts, among them U1 rp2040-zero

Commit message: added full version
Other:
- moved on the sheet: BZ1, R5
Changed lines of the file:
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@@
+	(wire
+		(pts
+			(xy 143.51 90.17) (xy 139.7 90.17)
+		)
+		(stroke
+			(width 0)
+			(type default)
+		)
+	)
+	(wire
+		(pts
+			(xy 153.67 92.71) (xy 156.21 92.71)
+		)
+		(stroke
+			(width 0)
+			(type default)
+		)
+	)
 	(wire
 		(pts
@@
 	(wire
 		(pts
-			(xy 142.24 95.25) (xy 156.21 95.25)
+			(xy 142.24 97.79) (xy 156.21 97.79)
 		)
 		(stroke
@@
 	(wire
 		(pts
-			(xy 142.24 95.25) (xy 142.24 99.06)
+			(xy 142.24 97.79) (xy 142.24 99.06)
 		)
 		(stroke
@@
 	(wire
 		(pts
-			(xy 144.78 90.17) (xy 139.7 90.17)
+			(xy 144.78 95.25) (xy 143.51 95.25)
+		)
+		(stroke
+			(width 0)
+			(type default)
+		)
+	)
+	(wire
+		(pts
+			(xy 153.67 95.25) (xy 153.67 92.71)
 		)
 		(stroke
@@
 	(wire
 		(pts
-			(xy 156.21 90.17) (xy 152.4 90.17)
+			(xy 143.51 95.25) (xy 143.51 90.17)
+		)
+		(stroke
+			(width 0)
+			(type default)
+		)
+	)
+	(wire
+		(pts
+			(xy 153.67 95.25) (xy 152.4 95.25)
 		)
 		(stroke
@@
 	(symbol
 		(lib_id "Device:R")
-		(at 148.59 90.17 90)
+		(at 148.59 95.25 90)
 		(unit 1)
 		(exclude_from_sim no)
@@
 		(dnp no)
 		(property "Reference" "R5"
-			(at 148.59 85.344 90)
+			(at 148.59 90.424 90)
 			(effects
 				(font
@@
 		)
 		(property "Value" "220 Ω"
-			(at 148.59 87.884 90)
+			(at 148.59 92.964 90)
 			(effects
 				(font
@@
 		)
 		(property "Footprint" "Resistor_SMD:R_1206_3216Metric_Pad1.30x1.75mm_HandSolder"
-			(at 148.59 91.948 90)
+			(at 148.59 97.028 90)
 			(effects
 				(font
@@
 		)
 		(property "Datasheet" "~"
-			(at 148.59 90.17 0)
+			(at 148.59 95.25 0)
 			(effects
 				(font
@@
 		)
 		(property "Description" "Resistor"
-			(at 148.59 90.17 0)
+			(at 148.59 95.25 0)
 			(effects
 				(font
@@
 	(symbol
 		(lib_id "Device:Buzzer")
-		(at 158.75 92.71 0)
+		(at 158.75 95.25 0)
 		(unit 1)
 		(exclude_from_sim no)
@@
 		(dnp no)
 		(property "Reference" "BZ1"
-			(at 162.56 91.4399 0)
+			(at 162.56 93.9799 0)
 			(effects
 				(font
@@
 		)
 		(property "Value" "Buzzer"
-			(at 162.56 93.9799 0)
+			(at 162.56 96.5199 0)
 			(effects
 				(font
@@
 		)
 		(property "Footprint" "Buzzer_Beeper:Buzzer_12x9.5RM7.6"
-			(at 158.115 90.17 90)
+			(at 158.115 92.71 90)
 			(effects
 				(font
@@
 		)
 		(property "Datasheet" "~"
-			(at 158.115 90.17 90)
+			(at 158.115 92.71 90)
 			(effects
 				(font
@@
 		)
 		(property "Description" "Buzzer, polarized"
-			(at 158.75 92.71 0)
-			(effects
-				(font
+			(at 158.75 95.25 0)
+			(effects
+				(font
