File: pcb/pcb/pcb.kicad_pcb (KiCad board)
At the start: 2 copper layers, 41 x 41 mm, 14 parts, among them U1 rp2040-zero

Commit message: added gerber files
Parts:
- added G***: LOGO, LOGO, B.Cu at (150.0, 50.0)
- added keychain1: MountingHole, MountingHole:MountingHole_3.2mm_M3, F.Cu at (133.0, 33.0)
Routing:
- net GND: track 0.00 -> 101.4 mm, vias 0 -> 4
- net Net-(U1-5): track 0.00 -> 53.9 mm
- net Net-(U1-3): track 0.00 -> 42.4 mm, vias 0 -> 1
- net Net-(U1-10): track 0.00 -> 39.5 mm, vias 0 -> 3
- net Net-(U1-11): track 0.00 -> 32.0 mm
- net Net-(U1-2): track 0.00 -> 27.4 mm, vias 0 -> 1
- net Net-(U1-12): track 0.00 -> 25.1 mm, vias 0 -> 2
- net Net-(BZ1-+): track 0.00 -> 21.3 mm, vias 0 -> 3
- net Net-(U1-13): track 0.00 -> 13.1 mm, vias 0 -> 2
- net Net-(U1-4): track 0.00 -> 7.88 mm
- net Net-(TR1-A): track 0.00 -> 2.53 mm
- net Net-(TL1-A): track 0.00 -> 2.53 mm
- net Net-(BR1-A): track 0.00 -> 2.53 mm
- net Net-(BL1-A): track 0.00 -> 2.51 mm
Other:
- outline, holes or cut-outs redrawn
- board text added: "COLOR_REPETER"
- board text added: "gaetancantelobre@github 10/24"

Commit message: added full version
Parts:
- added R5: 220 Ω, Resistor_SMD:R_1206_3216Metric_Pad1.30x1.75mm_HandSolder, F.Cu at (159.0, 65.5)
- moved G*** 1.21 mm to (149.7, 51.2)
Connections:
- U1 pad 7: Net-(BZ1-+) -> Net-(U1-6)
Routing:
- net Net-(U1-6): track 0.00 -> 22.2 mm, vias 0 -> 3
- net Net-(BZ1-+): track 21.3 -> 12.5 mm, vias 3 -> 0
Other:
- board text added: "->"
- board text added: "BEEP"
- board text added: "Simon Game Clone"
- board text added: "TWIM"
- board text removed: "COLOR_REPETER"
